File: ditto.kicad_sch (KiCad schematic)
At the start: 136 parts, among them J2 USB_C_Receptacle_USB2.0, SW1 SW_Push, SW10 SW_Push, SW11 SW_Push, SW12 SW_Push, SW13 SW_Push, SW14 SW_Push, SW15 SW_Push, SW16 SW_Push, SW17 SW_Push, SW18 SW_Push, SW19 SW_Push, SW2 SW_Push, SW20 SW_Push, SW21 SW_Push, SW22 SW_Push, SW23 SW_Push, SW24 SW_Push, SW25 SW_Push, SW26 SW_Push, SW27 SW_Push, SW28 SW_Push, SW29 SW_Push, SW3 SW_Push, SW30 SW_Push, SW31 SW_Push, SW32 SW_Push, SW33 SW_Push, SW34 SW_Push, SW35 SW_Push, SW36 SW_Push, SW37 SW_Push, SW38 SW_Push, SW39 SW_Push, SW4 SW_Push, SW40 SW_Push, SW5 SW_Push, SW6 SW_Push, SW7 SW_Push, SW8 SW_Push, SW9 SW_Push, U1 RP2040, U2 AP2112K-3.3, U3 W25Q128JVS, Y1 Crystal_GND24

Commit message: added logic level shifter for neopixels, gerbers, 3d file
Parts:
- added U3: SN74AHCT125QDRG4Q1, dip:SN74AHCT125QDRG4Q1, symbol 2022-05-06_03-58-36:SN74AHCT125QDRG4Q1
- C17, C18: value (none) -> 1µ
- C19, C20, C21: value (none) -> 10µ
- C25: value (none) -> 2.2µ
- H1: value (none) -> MountingHole; footprint (none) -> MountingHole:MountingHole_2.2mm_M2_DIN965_Pad
- H2, H3, H4: footprint (none) -> MountingHole:MountingHole_2.2mm_M2_DIN965_Pad
- J1: value (none) -> Conn_01x21; footprint (none) -> Connector_PinHeader_1.00mm:PinHeader_1x22_P1.00mm_Horizontal
- R10: value (none) -> 200
- R13: value (none) -> 1
- renumbered U3 to U4
Connections:
- net +5V: now also U3.14 (VCC)
- net GND: now also U3.1 (*1OE), U3.4 (*2OE), U3.7 (GND)
- net LEDS: now also U3.2 (1A); no longer R1.2
- new net LEDS_5V: R1.2, U3.3 (1Y)
- no-connect marks 2 -> 10
