File: electrical/ditto.kicad_pcb (KiCad board)
At the start: 2 copper layers, 257 x 91 mm, 137 parts, among them J1 Conn_01x21, J2 USB_C_Receptacle_USB2.0, SW1 SW_Push, SW10 SW_Push, SW11 SW_Push, SW12 SW_Push, SW13 SW_Push, SW14 SW_Push, SW15 SW_Push, SW16 SW_Push, SW17 SW_Push, SW18 SW_Push, SW19 SW_Push, SW2 SW_Push, SW20 SW_Push, SW21 SW_Push, SW22 SW_Push, SW23 SW_Push, SW24 SW_Push, SW25 SW_Push, SW26 SW_Push, SW27 SW_Push, SW28 SW_Push, SW29 SW_Push, SW3 SW_Push, SW30 SW_Push, SW31 SW_Push, SW32 SW_Push, SW33 SW_Push, SW34 SW_Push, SW35 SW_Push, SW36 SW_Push, SW37 SW_Push, SW38 SW_Push, SW39 SW_Push, SW4 SW_Push, SW40 SW_Push, SW5 SW_Push, SW6 SW_Push, SW7 SW_Push, SW8 SW_Push, SW9 SW_Push, U1 RP2040, U2 AP2112K-3.3, U3 SN74AHCT125QDRG4Q1, U4 W25Q128JVS, Y1 Crystal_GND24

Commit message: PDFs
Parts:
- moved C12 107.2 mm to (76.1, 55.1)
- moved D10 107.2 mm to (138.0, 55.4)
- moved D11 107.2 mm to (153.0, 55.4)
- moved D12 107.2 mm to (164.2, 55.4)
- moved D13 107.2 mm to (175.4, 55.4)
- moved D15 107.2 mm to (201.6, 55.4)
- moved D16 107.2 mm to (212.9, 55.4)
- moved D19 107.2 mm to (246.5, 55.4)
- moved D20 107.2 mm to (115.5, 55.4)
- moved D21 107.2 mm to (130.5, 55.4)
- moved D23 107.2 mm to (156.7, 55.4)
- moved D25 107.2 mm to (179.2, 55.4)
- moved D26 107.2 mm to (194.1, 55.4)
- moved D27 107.2 mm to (205.4, 55.4)
- moved D3 107.2 mm to (76.1, 59.1)
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